File: KiCad/PowerSupplies/PowerSupplies.sch (KiCad schematic (older format))
At the start: 6 parts

Commit message: 1-20-23
Parts:
- added 10V: D_Zener, symbol Device:D_Zener
- added C1: 1000uF, symbol Device:CP1
- added D1, D2: DIODE, symbol Simulation_SPICE:DIODE
- added RL: min100Ω, symbol Device:R_US
- added RS: 91Ω, symbol Device:R_US
- added T?: Transformer_1P_SS, symbol Device:Transformer_1P_SS
- gave numbers to parts that had none: 3
Connections:
- wire segments 16 -> 44
