File: KiCad/PowerSupplies/PowerSupplies.kicad_sch (KiCad schematic)
At the start: 54 parts, among them M1 Servo_9G, M1 Stepper_Motor_unipolar_5pin, M2 Servo_9G, SW1 SW_Push, U1 8x8 Dot Matrix, U1 HC-SR04, U1 MMA8452Q, U1 Stepper_Driver_IC, U2 Joystick, U2 PIR Motion Sensor

Commit message: update
Parts:
- added U2: 8x8 Dot Matrix, Package_DFN_QFN:DFN-8-1EP_2x2mm_P0.5mm_EP0.9x1.5mm, symbol Sensor_Touch:AT42QT1010-M
Connections:
- net +5V: now also U2. (V)
- net +VDC: now also U2. (V)
- net at A1_Nano1.23 (A4), U1. (VCC): now also U2. (V)
- net at A1_Nano1.24 (A5), U1. (VCC): now also U2. (V)
- new net: M1., U1. (Y) (x4)
Other:
- moved on the sheet: U1
Changed lines of the file:
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@@
   (junction (at 161.29 25.4) (diameter 0) (color 0 0 0 0)
   )
+  (junction (at 93.98 381) (diameter 0) (color 0 0 0 0)
+  )
   (junction (at 125.73 74.93) (diameter 0) (color 0 0 0 0)
   )
@@
   (junction (at 252.73 143.51) (diameter 0) (color 0 0 0 0)
   )
+  (junction (at 96.52 383.54) (diameter 0) (color 0 0 0 0)
+  )
   (junction (at 256.54 120.65) (diameter 0) (color 0 0 0 0)
   )
@@
     (stroke (width 0) (type default) (color 0 0 0 0))
   )
-  (wire (pts (xy 93.98 368.3) (xy 93.98 381))
+  (wire (pts (xy 93.98 353.06) (xy 93.98 381))
     (stroke (width 0) (type default) (color 0 0 0 0))
   )
@@
     (stroke (width 0) (type default) (color 0 0 0 0))
   )
+  (wire (pts (xy 96.52 383.54) (xy 96.52 388.62))
+    (stroke (width 0) (type default) (color 0 0 0 0))
+  )
   (wire (pts (xy 184.15 87.63) (xy 171.45 87.63))
     (stroke (width 0) (type default) (color 0 0 0 0))
@@
     (stroke (width 0) (type default) (color 0 0 0 0))
   )
+  (wire (pts (xy 99.06 386.08) (xy 93.98 386.08))
+    (stroke (width 0) (type default) (color 0 0 0 0))
+  )
   (wire (pts (xy 125.73 76.2) (xy 125.73 74.93))
     (stroke (width 0) (type default) (color 0 0 0 0))
@@
     (stroke (width 0) (type default) (color 0 0 0 0))
   )
+  (wire (pts (xy 96.52 355.6) (xy 99.06 355.6))
+    (stroke (width 0) (type default) (color 0 0 0 0))
+  )
   (wire (pts (xy 245.11 143.51) (xy 252.73 143.51))
     (stroke (width 0) (type default) (color 0 0 0 0))
@@
     (stroke (width 0) (type default) (color 0 0 0 0))
   )
-  (wire (pts (xy 96.52 370.84) (xy 96.52 383.54))
+  (wire (pts (xy 96.52 355.6) (xy 96.52 383.54))
     (stroke (width 0) (type default) (color 0 0 0 0))
   )
@@
     (stroke (width 0) (type default) (color 0 0 0 0))
   )
-  (wire (pts (xy 109.22 360.68) (xy 109.22 345.44))
+  (wire (pts (xy 269.24 66.04) (xy 269.24 67.31))
     (stroke (width 0) (type default) (color 0 0 0 0))
   )
-  (wire (pts (xy 269.24 66.04) (xy 269.24 67.31))
+  (wire (pts (xy 93.98 386.08) (xy 93.98 381))
+    (stroke (width 0) (type default) (color 0 0 0 0))
+  )
+  (wire (pts (xy 96.52 388.62) (xy 99.06 388.62))
     (stroke (width 0) (type default) (color 0 0 0 0))
   )
@@
     (stroke (width 0) (type default) (color 0 0 0 0))
   )
+  (wire (pts (xy 93.98 353.06) (xy 99.06 353.06))
+    (stroke (width 0) (type default) (color 0 0 0 0))
+  )
   (wire (pts (xy 422.91 175.26) (xy 426.72 175.26))
     (stroke (width 0) (type default) (color 0 0 0 0))
@@
     (stroke (width 0) (type default) (color 0 0 0 0))
   )
-  (wire (pts (xy 99.06 368.3) (xy 93.98 368.3))
-    (stroke (width 0) (type default) (color 0 0 0 0))
-  )
   (wire (pts (xy 261.62 143.51) (xy 261.62 140.97))
     (stroke (width 0) (type default) (color 0 0 0 0))
@@
     (stroke (width 0) (type default) (color 0 0 0 0))
   )
-  (wire (pts (xy 99.06 370.84) (xy 96.52 370.84))
-    (stroke (width 0) (type default) (color 0 0 0 0))
-  )
   (wire (pts (xy 245.11 130.81) (xy 250.19 130.81))
     (stroke (width 0) (type default) (color 0 0 0 0))
@@
     (pin "1")
   )
+  (symbol (lib_id "power:+5V") (at 109.22 378.46 0) (mirror y) (unit 1)
+    (in_bom yes) (on_board yes) (fields_autoplaced)
+    (property "Reference" "#PWR?" (id 0) (at 109.22 382.27 0)
+      (effects (font (size 1.27 1.27)) hide)
+    )
+    (property "Value" "+5V" (id 1) (at 109.22 373.38 0))
+    (property "Footprint" "" (id 2) (at 109.22 378.46 0)
+      (effects (font (size 1.27 1.27)) hide)
+    )
+    (property "Datasheet" "" (id 3) (at 109.22 378.46 0)
+      (effects (font (size 1.27 1.27)) hide)
+    )
+    (pin "1")
+  )
   (symbol (lib_id "Device:R_Potentiometer_US") (at 444.5 217.17 0) (mirror x) (unit 1)
     (in_bom yes) (on_board yes)
@@
     (pin "2")
   )
-  (symbol (lib_id "power:GND") (at 109.22 378.46 0) (unit 1)
+  (symbol (lib_id "power:GND") (at 109.22 396.24 0) (unit 1)
     (in_bom yes) (on_board yes) (fields_autoplaced)
-    (property "Reference" "#PWR?" (id 0) (at 109.22 384.81 0)
+    (property "Reference" "#PWR?" (id 0) (at 109.22 402.59 0)
       (effects (font (size 1.27 1.27)) hide)
     )
-    (property "Value" "GND" (id 1) (at 109.22 383.54 0))
-    (property "Footprint" "" (id 2) (at 109.22 378.46 0)
+    (property "Value" "GND" (id 1) (at 109.22 401.32 0))
+    (property "Footprint" "" (id 2) (at 109.22 396.24 0)
       (effects (font (size 1.27 1.27)) hide)
     )
-    (property "Datasheet" "" (id 3) (at 109.22 378.46 0)
+    (property "Datasheet" "" (id 3) (at 109.22 396.24 0)
       (effects (font (size 1.27 1.27)) hide)
     )
@@
     (pin "1")
   )
+  (symbol (lib_id "power:GND") (at 109.22 363.22 0) (unit 1)
+    (in_bom yes) (on_board yes) (fields_autoplaced)
+    (property "Reference" "#PWR?" (id 0) (at 109.22 369.57 0)
+      (effects (font (size 1.27 1.27)) hide)
+    )
+    (property "Value" "GND" (id 1) (at 109.22 368.3 0))
+    (property "Footprint" "" (id 2) (at 109.22 363.22 0)
+      (effects (font (size 1.27 1.27)) hide)
+    )
+    (property "Datasheet" "" (id 3) (at 109.22 363.22 0)
+      (effects (font (size 1.27 1.27)) hide)
+    )
+    (pin "1")
+  )
+  (symbol (lib_name "AT42QT1010-M_4") (lib_id "Sensor_Touch:AT42QT1010-M") (at 109.22 386.08 0) (unit 1)
+    (in_bom yes) (on_board yes)
+    (property "Reference" "U2" (id 0) (at 114.3 377.19 0)
+      (effects (font (size 1.27 1.27)) (justify right))
+    )
+    (property "Value" "8x8 Dot Matrix" (id 1) (at 125.73 379.73 0)
+      (effects (font (size 1.27 1.27)) (justify right))
+    )
+    (property "Footprint" "Package_DFN_QFN:DFN-8-1EP_2x2mm_P0.5mm_EP0.9x1.5mm" (id 2) (at 110.49 394.97 0)
+      (effects (font (size 1.27 1.27)) (justify left) hide)
+    )
+    (property "Datasheet" "http://ww1.microchip.com/downloads/en/DeviceDoc/40001946A.pdf" (id 3) (at 116.078 372.11 0)
+      (effects (font (size 1.27 1.27)) hide)
+    )
+    (pin "")
+    (pin "")
+    (pin "")
+    (pin "")
+    (pin "")
+  )
   (symbol (lib_id "power:+5V") (at 392.43 218.44 0) (unit 1)
     (in_bom yes) (on_board yes) (fields_autoplaced)
@@
     (pin "2")
   )
-  (symbol (lib_name "AT42QT1010-M_5") (lib_id "Sensor_Touch:AT42QT1010-M") (at 109.22 368.3 0) (unit 1)
+  (symbol (lib_name "AT42QT1010-M_5") (lib_id "Sensor_Touch:AT42QT1010-M") (at 109.22 353.06 0) (unit 1)
     (in_bom yes) (on_board yes)
-    (property "Reference" "U1" (id 0) (at 114.3 359.41 0)
+    (property "Reference" "U1" (id 0) (at 114.3 344.17 0)
       (effects (font (size 1.27 1.27)) (justify right))
     )
-    (property "Value" "MMA8452Q" (id 1) (at 121.92 361.95 0)
+    (property "Value" "MMA8452Q" (id 1) (at 121.92 346.71 0)
       (effects (font (size 1.27 1.27)) (justify right))
     )
-    (property "Footprint" "Package_DFN_QFN:DFN-8-1EP_2x2mm_P0.5mm_EP0.9x1.5mm" (id 2) (at 110.49 377.19 0)
+    (property "Footprint" "Package_DFN_QFN:DFN-8-1EP_2x2mm_P0.5mm_EP0.9x1.5mm" (id 2) (at 110.49 361.95 0)
       (effects (font (size 1.27 1.27)) (justify left) hide)
     )
-    (property "Datasheet" "http://ww1.microchip.com/downloads/en/DeviceDoc/40001946A.pdf" (id 3) (at 116.078 354.33 0)
+    (property "Datasheet" "http://ww1.microchip.com/downloads/en/DeviceDoc/40001946A.pdf" (id 3) (at 116.078 339.09 0)
       (effects (font (size 1.27 1.27)) hide)
     )
@@
       (reference "#PWR?") (unit 1) (value "GND") (footprint "")
     )
+    (path "/8dafb83f-62ee-4487-aa22-d274f56644b4"
+      (reference "#PWR?") (unit 1) (value "+5V") (footprint "")
+    )
     (path "/94f5438c-fa31-4025-97ec-22c58c609c4f"
       (reference "#PWR?") (unit 1) (value "GND") (footprint "")
@@
       (reference "#PWR?") (unit 1) (value "GND") (footprint "")
     )
+    (path "/d33e9e0e-011a-461b-bc1e-177371bf6b94"
+      (reference "#PWR?") (unit 1) (value "GND") (footprint "")
+    )
     (path "/da133c39-4aa2-4c5f-b0fd-f9eee112b966"
       (reference "#PWR?") (unit 1) (value "+5V") (footprint "")
@@
       (reference "U1") (unit 1) (value "MMA8452Q") (footprint "Package_DFN_QFN:DFN-8-1EP_2x2mm_P0.5mm_EP0.9x1.5mm")
     )
+    (path "/d9772f5a-4f30-450c-a84d-b6aa35d18462"
+      (reference "U2") (unit 1) (value "8x8 Dot Matrix") (footprint "Package_DFN_QFN:DFN-8-1EP_2x2mm_P0.5mm_EP0.9x1.5mm")
+    )
     (path "/ef57a7fe-9cc8-4852-879c-ebdff2f9f147"
