File: KiCad/Amplifiers/LM1875/LM1875/_autosave-LM1875.kicad_pcb (KiCad board)
At the start: 2 copper layers, 125.1 x 70 mm, 42 parts, among them J1 Screw_Terminal_01x04, J2 AudioJack3, U1 LM1875, U2 LM1875

Commit message: update
Parts:
- moved H4 159.4 mm to (204.2, 61.3)
- moved J2 157.8 mm to (88.6, 111.1)
- moved C1 156.6 mm to (125.6, 80.6)
- moved C10 156.6 mm to (164.7, 83.1)
- moved C11 156.6 mm to (122.5, 61.3)
- moved C12 156.6 mm to (151.7, 61.3)
- moved C13 156.6 mm to (176.4, 83.7)
- moved C14 156.6 mm to (176.4, 107.5)
- moved C2 156.6 mm to (134.1, 80.6)
- moved C3 156.6 mm to (142.6, 80.6)
- moved C4 156.6 mm to (107.1, 83.1)
- moved C5 156.6 mm to (151.1, 80.6)
- moved C6 156.6 mm to (116.0, 83.1)
- moved C7 156.6 mm to (114.0, 63.8)
- moved C8 156.6 mm to (143.5, 63.8)
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Other:
- board size 125.1 x 70 mm -> 126.2 x 69.8 mm
