File: KiCad/Amplifiers/LM1875/LM1875/_autosave-LM1875.kicad_sch (KiCad schematic)
At the start: 42 parts, among them J2 Screw_Terminal_01x04, J3 AudioJack3, U1 LM1875, U2 LM1875

Commit message: update
Parts:
- removed R11, R12: 100K, Potentiometer_THT:Potentiometer_Alps_RK163_Single_Horizontal, symbol Device:R_Variable_US
- added R11, R12: 100K, Resistor_THT:R_Axial_DIN0309_L9.0mm_D3.2mm_P12.70mm_Horizontal, symbol Device:R_Small_US
- renumbered J2 to J1, J3 to J2
Connections:
- net at R5.2, U1.2 (-): now also R11.1
- net at R15.1: now also R11.2
- net at R6.2, U2.2 (-): now also R12.1
- net at R16.1: now also R12.2
Changed lines of the file:
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@@
     (stroke (width 0) (type default) (color 0 0 0 0))
   )
-  (wire (pts (xy 144.78 152.4) (xy 148.59 152.4))
+  (wire (pts (xy 144.78 152.4) (xy 149.86 152.4))
     (stroke (width 0) (type default) (color 0 0 0 0))
   )
@@
     (stroke (width 0) (type default) (color 0 0 0 0))
   )
-  (wire (pts (xy 156.21 152.4) (xy 165.1 152.4))
+  (wire (pts (xy 154.94 152.4) (xy 165.1 152.4))
     (stroke (width 0) (type default) (color 0 0 0 0))
   )
@@
     (stroke (width 0) (type default) (color 0 0 0 0))
   )
-  (wire (pts (xy 154.94 99.06) (xy 163.83 99.06))
+  (wire (pts (xy 153.67 99.06) (xy 163.83 99.06))
     (stroke (width 0) (type default) (color 0 0 0 0))
   )
@@
     (stroke (width 0) (type default) (color 0 0 0 0))
   )
-  (wire (pts (xy 143.51 99.06) (xy 147.32 99.06))
+  (wire (pts (xy 143.51 99.06) (xy 148.59 99.06))
     (stroke (width 0) (type default) (color 0 0 0 0))
   )
@@
     )
   )
+  (symbol (lib_id "Device:R_Small_US") (at 151.13 99.06 90) (unit 1)
+    (in_bom yes) (on_board yes)
+    (property "Reference" "R11" (id 0) (at 151.13 93.98 90))
+    (property "Value" "100K" (id 1) (at 151.13 96.52 90))
+    (property "Footprint" "Resistor_THT:R_Axial_DIN0309_L9.0mm_D3.2mm_P12.70mm_Horizontal" (id 2) (at 151.13 99.06 0)
+      (effects (font (size 1.27 1.27)) hide)
+    )
+    (property "Datasheet" "~" (id 3) (at 151.13 99.06 0)
+      (effects (font (size 1.27 1.27)) hide)
+    )
+    (pin "1")
+    (pin "2")
+  )
   (symbol (lib_id "power:GND") (at 151.13 88.9 0) (unit 1)
     (in_bom yes) (on_board yes)
@@
     )
     (property "Datasheet" "~" (id 3) (at 128.27 101.6 0)
-      (effects (font (size 1.27 1.27)) hide)
-    )
-    (pin "1")
-    (pin "2")
-  )
-  (symbol (lib_id "Device:R_Variable_US") (at 151.13 99.06 90) (unit 1)
-    (in_bom yes) (on_board yes)
-    (property "Reference" "R11" (id 0) (at 151.13 92.71 90))
-    (property "Value" "100K" (id 1) (at 151.13 95.25 90))
-    (property "Footprint" "Potentiometer_THT:Potentiometer_Alps_RK163_Single_Horizontal" (id 2) (at 151.13 100.838 90)
-      (effects (font (size 1.27 1.27)) hide)
-    )
-    (property "Datasheet" "~" (id 3) (at 151.13 99.06 0)
       (effects (font (size 1.27 1.27)) hide)
     )
@@
   (symbol (lib_id "Connector:AudioJack3") (at 99.06 91.44 0) (unit 1)
     (in_bom yes) (on_board yes) (fields_autoplaced)
-    (property "Reference" "J3" (id 0) (at 97.155 82.55 0))
+    (property "Reference" "J2" (id 0) (at 97.155 82.55 0))
     (property "Value" "AudioJack3" (id 1) (at 97.155 85.09 0))
     (property "Footprint" "Connector_Audio:Jack_3.5mm_CUI_SJ1-3525N_Horizontal" (id 2) (at 99.06 91.44 0)
@@
     (pin "2")
   )
-  (symbol (lib_id "Device:R_Variable_US") (at 152.4 152.4 90) (unit 1)
-    (in_bom yes) (on_board yes)
-    (property "Reference" "R12" (id 0) (at 152.4 146.05 90))
-    (property "Value" "100K" (id 1) (at 152.4 148.59 90))
-    (property "Footprint" "Potentiometer_THT:Potentiometer_Alps_RK163_Single_Horizontal" (id 2) (at 152.4 154.178 90)
+  (symbol (lib_id "Device:R_Small_US") (at 152.4 152.4 90) (unit 1)
+    (in_bom yes) (on_board yes)
+    (property "Reference" "R12" (id 0) (at 152.4 147.32 90))
+    (property "Value" "100K" (id 1) (at 152.4 149.86 90))
+    (property "Footprint" "Resistor_THT:R_Axial_DIN0309_L9.0mm_D3.2mm_P12.70mm_Horizontal" (id 2) (at 152.4 152.4 0)
       (effects (font (size 1.27 1.27)) hide)
     )
@@
   (symbol (lib_id "Connector:Screw_Terminal_01x04") (at 96.52 71.12 0) (mirror y) (unit 1)
     (in_bom yes) (on_board yes) (fields_autoplaced)
-    (property "Reference" "J2" (id 0) (at 96.52 62.23 0))
+    (property "Reference" "J1" (id 0) (at 96.52 62.23 0))
     (property "Value" "Screw_Terminal_01x04" (id 1) (at 96.52 64.77 0))
     (property "Footprint" "TerminalBlock_Phoenix:TerminalBlock_Phoenix_MKDS-1,5-4_1x04_P5.00mm_Horizontal" (id 2) (at 96.52 71.12 0)
@@
     )
     (path "/fdb54752-5dff-4aca-987f-2aee2ebf8590"
-      (reference "J2") (unit 1) (value "Screw_Terminal_01x04") (footprint "TerminalBlock_Phoenix:TerminalBlock_Phoenix_MKDS-1,5-4_1x04_P5.00mm_Horizontal")
+      (reference "J1") (unit 1) (value "Screw_Terminal_01x04") (footprint "TerminalBlock_Phoenix:TerminalBlock_Phoenix_MKDS-1,5-4_1x04_P5.00mm_Horizontal")
     )
     (path "/4d06b349-705d-4cf9-a596-1252a5486135"
-      (reference "J3") (unit 1) (value "AudioJack3") (footprint "Connector_Audio:Jack_3.5mm_CUI_SJ1-3525N_Horizontal")
+      (reference "J2") (unit 1) (value "AudioJack3") (footprint "Connector_Audio:Jack_3.5mm_CUI_SJ1-3525N_Horizontal")
     )
     (path "/3540c8ff-f9cd-4d72-bad8-a85428a27567"
@@
       (reference "R10") (unit 1) (value "22K") (footprint "Resistor_THT:R_Axial_DIN0309_L9.0mm_D3.2mm_P12.70mm_Horizontal")
     )
-    (path "/34565911-1df0-4245-8d24-e48b2136fee3"
-      (reference "R11") (unit 1) (value "100K") (footprint "Potentiometer_THT:Potentiometer_Alps_RK163_Single_Horizontal")
-    )
-    (path "/8ccd102b-cb04-48af-a825-edd2632ffd01"
-      (reference "R12") (unit 1) (value "100K") (footprint "Potentiometer_THT:Potentiometer_Alps_RK163_Single_Horizontal")
+    (path "/00533118-67c8-4581-a79e-997ed264739c"
+      (reference "R11") (unit 1) (value "100K") (footprint "Resistor_THT:R_Axial_DIN0309_L9.0mm_D3.2mm_P12.70mm_Horizontal")
+    )
+    (path "/8cd93b97-0176-4e65-8be6-7434503b219f"
+      (reference "R12") (unit 1) (value "100K") (footprint "Resistor_THT:R_Axial_DIN0309_L9.0mm_D3.2mm_P12.70mm_Horizontal")
     )
     (path "/4b5aa05d-e28a-4abf-96b4-c552a769b65d"
